File: LED/led_v1/led_v1.kicad_sch (KiCad schematic)
At the start: 14 parts

Commit message: Send order for v1
Parts:
- added J2: Screw_Terminal_01x02, TerminalBlock_Phoenix:TerminalBlock_Phoenix_MKDS-1,5-2-5.08_1x02_P5.08mm_Horizontal, symbol Connector:Screw_Terminal_01x02
- C1: renamed from C?; JLC C28323 -> 0805; LCSC (none) -> C28323
- D1, D2, D3, D4, D5, D6: renamed from D?; JLC C83955 -> LED_0603; LCSC (none) -> C83955
- R1, R2, R3, R4, R5, R6: renamed from R?; JLC C25091 -> 0402; LCSC (none) -> C25091
- gave numbers to parts that had none: 1
Connections:
- net +5V: now reaches C1.2, J1.2 (Pin_2), R1.2, R2.2, R3.2, R4.2, R5.2, R6.2
- net +5V: now also J2.2 (Pin_2)
- net GNDREF: now reaches C1.1, D1.1 (K), D2.1 (K), D3.1 (K), D4.1 (K), D5.1 (K), D6.1 (K), J1.1 (Pin_1)
- net GNDREF: now also J2.1 (Pin_1)
